Commit message: fix: correct URDF mesh paths from ../../meshes/ to ../meshes/

File: czy/data/x1_29/urdf/X1_29DOF_perfect_mirrored.urdf (robot description, URDF)
Before this commit: robot x1, 60 links, 59 joints
Links:
- link arm_l_wrist_a_ball_link: geometry visual mesh filename=../meshes/arm_r_wrist_a_ball.STL
- link arm_l_wrist_a_loop_link: geometry visual mesh filename=../meshes/arm_r_wrist_a_loop.STL
- link arm_l_wrist_b_ball_link: geometry visual mesh filename=../meshes/arm_r_wrist_b_ball.STL
- link arm_l_wrist_b_loop_link: geometry visual mesh filename=../meshes/arm_r_wrist_b_loop.STL
- link arm_l_wrist_motor_a_link: geometry visual mesh filename=../meshes/arm_r_wrist_motor_a_link.STL
- link arm_l_wrist_motor_b_link: geometry visual mesh filename=../meshes/arm_r_wrist_motor_b_link.STL
- link arm_r_wrist_a_ball_link: geometry visual mesh filename=../meshes/arm_r_wrist_a_ball_right_perfect_mirrored.STL
- link arm_r_wrist_a_loop_link: geometry visual mesh filename=../meshes/arm_r_wrist_a_loop_right_perfect_mirrored.STL
- link arm_r_wrist_b_ball_link: geometry visual mesh filename=../meshes/arm_r_wrist_b_ball_right_perfect_mirrored.STL
- link arm_r_wrist_b_loop_link: geometry visual mesh filename=../meshes/arm_r_wrist_b_loop_right_perfect_mirrored.STL
- link arm_r_wrist_motor_a_link: geometry visual mesh filename=../meshes/arm_r_wrist_motor_a_link_right_perfect_mirrored.S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
- link arm_r_wrist_motor_b_link: geometry visual mesh filename=../meshes/arm_r_wrist_motor_a_link_perfect_mirrored.STL
- link base_link: geometry collision mesh filename=../meshes/base_link_simple_center_symmetric_collision.STL; visual mesh filename=../meshes/base_link_simple_center_symmetric.STL
- link left_ankle_pitch_link: geometry visual mesh filename=../meshes/left_ankle_pitch.STL
- link left_ankle_roll_link: geometry collision mesh filename=../meshes/left_ankle_roll.STL; visual mesh filename=../meshes/left_ankle_roll.STL
- link left_elbow_pitch_link: geometry visual mesh filename=../meshes/left_elbow_pitch.STL
- link left_elbow_yaw_link: geometry visual mesh filename=../meshes/left_elbow_yaw.STL
- link left_hip_pitch_link: geometry visual mesh filename=../meshes/left_hip_pitch.STL
- link left_hip_roll_link: geometry visual mesh filename=../meshes/left_hip_roll.STL
- link left_hip_yaw_link: geometry visual mesh filename=../meshes/left_hip_yaw.STL
- link left_knee_pitch_link: geometry visual mesh filename=../meshes/left_knee_pitch.STL
- link left_shoulder_pitch_link: geometry visual mesh filename=../meshes/left_shoulder_pitch.STL
- link left_shoulder_roll_link: geometry visual mesh filename=../meshes/left_shoulder_roll.STL
- link left_shoulder_yaw_link: geometry visual mesh filename=../meshes/left_shoulder_yaw.STL
- link left_wrist_pitch_link: geometry visual mesh filename=../meshes/left_wrist_pitch.STL
- link left_wrist_roll_link: geometry visual mesh filename=../meshes/left_wrist_roll.STL
- link leg_l_toe_a_ball_link: geometry visual mesh filename=../meshes/leg_l_toe_a_ball.STL
- link leg_l_toe_a_link: geometry visual mesh filename=../meshes/leg_l_toe_a_link.STL
- link leg_l_toe_a_loop_link: geometry visual mesh filename=../meshes/leg_l_toe_a_loop.STL
- link leg_l_toe_b_ball_link: geometry visual mesh filename=../meshes/leg_l_toe_b_ball.STL
- link leg_l_toe_b_link: geometry visual mesh filename=../meshes/leg_l_toe_b_link.STL
- link leg_l_toe_b_loop_link: geometry visual mesh filename=../meshes/leg_l_toe_b_loop.STL
- link leg_r_toe_a_ball_link: geometry visual mesh filename=../meshes/leg_r_toe_a_ball_perfect_mirrored.STL
- link leg_r_toe_a_link: geometry visual mesh filename=../meshes/leg_r_toe_a_link_perfect_mirrored.STL
- link leg_r_toe_a_loop_link: geometry visual mesh filename=../meshes/leg_r_toe_a_loop_perfect_mirrored.STL
- link leg_r_toe_b_ball_link: geometry visual mesh filename=../meshes/leg_r_toe_b_ball_perfect_mirrored.STL
- link leg_r_toe_b_link: geometry visual mesh filename=../meshes/leg_r_toe_b_link_perfect_mirrored.STL
- link leg_r_toe_b_loop_link: geometry visual mesh filename=../meshes/leg_r_toe_b_loop_perfect_mirrored.STL
- link lumbar_pitch_link: geometry visual mesh filename=../meshes/lumbar_pitch_x1_center_symmetric.STL
- link lumbar_roll_link: geometry visual mesh filename=../meshes/lumbar_roll_center_symmetric.STL
- link lumbar_yaw_link: geometry visual mesh filename=../meshes/lumbar_yaw_center_symmetric.STL
- link right_ankle_pitch_link: geometry visual mesh filename=../meshes/right_ankle_pitch_perfect_mirrored.STL
- link right_ankle_roll_link: geometry collision mesh filename=../meshes/right_ankle_roll_perfect_mirrored.STL; visual mesh filename=../meshes/right_ankle_roll_perfect_mirrored.STL
- link right_elbow_pitch_link: geometry visual mesh filename=../meshes/right_elbow_pitch_perfect_mirrored.STL
- link right_elbow_yaw_link: geometry visual mesh filename=../meshes/right_elbow_yaw_perfect_mirrored.STL
- link right_hip_pitch_link: geometry visual mesh filename=../meshes/right_hip_pitch_perfect_mirrored.STL
- link right_hip_roll_link: geometry visual mesh filename=../meshes/right_hip_roll_perfect_mirrored.STL
- link right_hip_yaw_link: geometry visual mesh filename=../meshes/right_hip_yaw_perfect_mirrored.STL
- link right_knee_pitch_link: geometry visual mesh filename=../meshes/right_knee_pitch_perfect_mirrored.STL
- link right_shoulder_pitch_link: geometry visual mesh filename=../meshes/right_shoulder_pitch_perfect_mirrored.STL
- link right_shoulder_roll_link: geometry visual mesh filename=../meshes/right_shoulder_roll_perfect_mirrored.STL
- link right_shoulder_yaw_link: geometry visual mesh filename=../meshes/right_shoulder_yaw_perfect_mirrored.STL
- link right_wrist_pitch_link: geometry visual mesh filename=../meshes/right_wrist_pitch_perfect_mirrored.STL
- link right_wrist_roll_link: geometry visual mesh filename=../meshes/right_wrist_roll_perfect_mirrored.STL
- link waist_motor_a_ball_link: geometry visual mesh filename=../meshes/waist_motor_a_ball_perfect_mirrored.STL
- link waist_motor_a_link: geometry visual mesh filename=../meshes/waist_motor_a_link_perfect_mirrored.STL
- link waist_motor_a_loop_link: geometry visual mesh filename=../meshes/waist_motor_a_loop_perfect_mirrored.STL
- link waist_motor_b_ball_link: geometry visual mesh filename=../meshes/waist_motor_b_ball.STL
- link waist_motor_b_link: geometry visual mesh filename=../meshes/waist_motor_b_link.STL
- link waist_motor_b_loop_link: geometry visual mesh filename=../meshes/waist_motor_b_loop.STL
